File: RP2040.sch (KiCad schematic (older format))
At the start: 45 parts, among them J1 Conn_01x12_Male, J2 Qwiic, J3 Conn_01x12_Male, J4 Conn_01x04_Male, U1 3.3V, U2 RP2040, U3 WS2812-2020, U4 W25QXX128MBIT, Y1 12MHz

Commit message: fixed file naming
Parts:
- removed TP3: TEST-POINT3X5, SparkFun_ProMicro-RP2040:PAD.03X.05, symbol SparkFun_ProMicro-RP2040-eagle-import:TEST-POINT3X5
- C11, C13: symbol SparkFun_ProMicro-RP2040-eagle-import:15PF-0402T-50V-5% -> RP2040-rescue:15PF-0402T-50V-5%-SparkFun_ProMicro-RP2040-eagle-import
- C12, C14, C15, C16, C17, C18, C19, C29, C9: symbol SparkFun_ProMicro-RP2040-eagle-import:0.1UF-0402T-6.3V-10%-X7R -> RP2040-rescue:0.1UF-0402T-6.3V-10%-X7R-SparkFun_ProMicro-RP2040-eagle-import
- C20, C21, C22, C23: symbol SparkFun_ProMicro-RP2040-eagle-import:2.2UF-0402_TIGHT-10V-10%-X5R -> RP2040-rescue:2.2UF-0402_TIGHT-10V-10%-X5R-SparkFun_ProMicro-RP2040-eagle-import
- C6: symbol SparkFun_ProMicro-RP2040-eagle-import:1.0UF-0402T-16V-10% -> RP2040-rescue:1.0UF-0402T-16V-10%-SparkFun_ProMicro-RP2040-eagle-import
- C7, C8: symbol SparkFun_ProMicro-RP2040-eagle-import:10UF-0402T-6.3V-20% -> RP2040-rescue:10UF-0402T-6.3V-20%-SparkFun_ProMicro-RP2040-eagle-import
- D2: symbol SparkFun_ProMicro-RP2040-eagle-import:DIODE-SCHOTTKY-BAT60A -> RP2040-rescue:DIODE-SCHOTTKY-BAT60A-SparkFun_ProMicro-RP2040-eagle-import
- F1: symbol SparkFun_ProMicro-RP2040-eagle-import:PPTC_6V500MA -> RP2040-rescue:PPTC_6V500MA-SparkFun_ProMicro-RP2040-eagle-import
- J2: symbol SparkFun_ProMicro-RP2040-eagle-import:QWIIC_CONNECTORJS-1MM -> RP2040-rescue:QWIIC_CONNECTORJS-1MM-SparkFun_ProMicro-RP2040-eagle-import
- LED1: symbol SparkFun_ProMicro-RP2040-eagle-import:LED-RED0603 -> RP2040-rescue:LED-RED0603-SparkFun_ProMicro-RP2040-eagle-import
- R10, R11, R15: symbol SparkFun_ProMicro-RP2040-eagle-import:1KOHM-0402T-1_16W-1% -> RP2040-rescue:1KOHM-0402T-1_16W-1%-SparkFun_ProMicro-RP2040-eagle-import
- R12, R13: symbol SparkFun_ProMicro-RP2040-eagle-import:27OHM -> RP2040-rescue:27OHM-SparkFun_ProMicro-RP2040-eagle-import
- R14: symbol SparkFun_ProMicro-RP2040-eagle-import:200OHM-0402T-1_16W-1% -> RP2040-rescue:200OHM-0402T-1_16W-1%-SparkFun_ProMicro-RP2040-eagle-import
- R16, R2: symbol SparkFun_ProMicro-RP2040-eagle-import:10KOHM-0402T-1_16W-1% -> RP2040-rescue:10KOHM-0402T-1_16W-1%-SparkFun_ProMicro-RP2040-eagle-import
- R5, R7: symbol SparkFun_ProMicro-RP2040-eagle-import:2.2KOHM-0402T-1_16W-1% -> RP2040-rescue:2.2KOHM-0402T-1_16W-1%-SparkFun_ProMicro-RP2040-eagle-import
- S1, S2: symbol SparkFun_ProMicro-RP2040-eagle-import:MOMENTARY-SWITCH-SPST-SMD-4.6X2.8MM -> RP2040-rescue:MOMENTARY-SWITCH-SPST-SMD-4.6X2.8MM-SparkFun_ProMicro-RP2040-eagle-import
- TP1, TP2: symbol SparkFun_ProMicro-RP2040-eagle-import:TEST-POINT3X5 -> RP2040-rescue:TEST-POINT3X5-SparkFun_ProMicro-RP2040-eagle-import
- U1: symbol SparkFun_ProMicro-RP2040-eagle-import:V_REG_AP2112K-3.3V -> RP2040-rescue:V_REG_AP2112K-3.3V-SparkFun_ProMicro-RP2040-eagle-import
- U2: symbol SparkFun_ProMicro-RP2040-eagle-import:RP2040 -> RP2040-rescue:RP2040-SparkFun_ProMicro-RP2040-eagle-import
- U3: symbol SparkFun_ProMicro-RP2040-eagle-import:WS2812-2020 -> RP2040-rescue:WS2812-2020-SparkFun_ProMicro-RP2040-eagle-import
- U4: symbol SparkFun_ProMicro-RP2040-eagle-import:W25QXX128MBIT-6X5-SKINNY_CENTER -> RP2040-rescue:W25QXX128MBIT-6X5-SKINNY_CENTER-SparkFun_ProMicro-RP2040-eagle-import
- Y1: symbol SparkFun_ProMicro-RP2040-eagle-import:CRYSTAL-12MHZ -> RP2040-rescue:CRYSTAL-12MHZ-SparkFun_ProMicro-RP2040-eagle-import
